File: Electronic/Placa PCB/interstage_A1.sch (EAGLE design)
At the start: 32 parts, among them U1 328P, Y1 16MHz

Commit message: Placas PCB
Parts:
- removed C2: 22pF, resistor:C-EU025-025X050
- removed C3: 100nF, resistor:C-EU025-025X050
- removed ISP6: (no value), pinhead:PINHD-2X3
- removed JP7: (no value), pinhead:PINHD-1X6
- removed LED13: (no value), pinhead:PINHD-1X2
- removed OUT1, OUT2, OUT3, OUT4, SET_VCC, SET_VIN: (no value), pinhead:PINHD-1X3
- removed PMV16XNR, PMV16XNR1, PMV16XNR2, PMV16XNR3: (no value), zetex:NMOSSOT23
- removed R10, R4, R5, R6, R7, R8, R9: 330 Ohm, resistor:R-EU_0204/7
- removed R11, R12: 10kohm, resistor:R-EU_0204/7
- removed U$1: SUCHAI_STACKBREAKOUT, SUCHAI_PCB:SUCHAI_STACKBREAKOUT
- removed U1: 328P, SparkFun-IC-Microcontroller:ATMEGA328P_PDIP
- added BOOT_LOADER, FTDI: 0532610671, picoblade6:0532610671
- added C4, C5: 22pF, rcl:C-EUC0603K
- added I2C: 0532610471, 0532610471:0532610471
- added J1, J2: 0532611271, picoblade:0532611271
- added PAD1, PAD2, PAD3, PAD4, PAD5, PAD6, PAD7: WIREPADSMD1,27-254, wirepad:WIREPADSMD1,27-254
- added Q1: PMV16XNR, SamacSys_Parts:PMV16XNR
- added U2: ATMEGA328P_TQFP, SparkFun-IC-Microcontroller:ATMEGA328P_TQFP
- C1: value 22pF -> 100nF; device resistor:C-EU025-025X050 -> rcl:C-EUC0805K
- R1, R3: device resistor:R-EU_0204/7 -> rcl:R-EU_R1206
- R2: value 220 Ohm -> 330 Ohm; device resistor:R-EU_0204/7 -> rcl:R-EU_R1206
- Y1: device SparkFun-Clocks:CRYSTAL-16MHZPTH-HC49US -> SparkFun-Clocks:CRYSTAL-16MHZSMD-2X1.6
Connections:
- removed net 3.3V/VCC: U$1.170, U$1.196, U$1.66, U$1.92
- removed net 5V-MAIN: U$1.146, U$1.42
- removed net 5V/VCC: U$1.169, U$1.195, U$1.65, U$1.91
- removed net AGND: U$1.172, U$1.68
- removed net CAN-H: U$1.106, U$1.2
- removed net CAN-L: U$1.1, U$1.105
- removed net CLK-MAIN: U$1.11, U$1.115
- removed net CS-MAIN: U$1.142, U$1.38
- removed net CS_-MAIN: U$1.117, U$1.13, U$1.143, U$1.39
- removed net EPS-RX: U$1.200, U$1.96
- removed net EPS-TX: U$1.201, U$1.97
- removed net I2C-SCL[A]: U$1.110, U$1.6
- removed net I2C-SCL[B]: U$1.126, U$1.22
- removed net I2C-SDA[A]: U$1.109, U$1.5
- removed net I2C-SDA[B]: U$1.125, U$1.21
- removed net MISO-MAIN: U$1.141, U$1.37
- removed net MOSI-MAIN: U$1.116, U$1.12
- removed net N$10: OUT2.3, PMV16XNR2.D
- removed net N$11: OUT1.3, PMV16XNR3.D
- removed net N$12: OUT4.1, R7.2
- removed net N$13: R7.1, U1.PD2(INT0)
- removed net N$14: OUT3.1, R8.2
- removed net N$15: R8.1, U1.PD4(XCK/T0)
- removed net N$16: R9.1, U1.PD7(AIN1)
- removed net N$17: OUT2.1, R9.2
- removed net N$19: R10.1, U1.PB0(ICP)
- removed net N$3: PMV16XNR.G, R3.1, U1.PD6(AIN0)
- removed net N$5: PMV16XNR1.G, R4.1, U1.PB1(OC1A)
- removed net N$7: PMV16XNR3.G, R6.1, U1.PD3(INT1)
- removed net N$8: OUT4.3, PMV16XNR1.D
- removed net N$9: OUT3.3, PMV16XNR.D
- removed net OUT1-3.3V: U$1.128, U$1.24
- removed net OUT2-3.3V: SET_VCC.3, SET_VIN.3, U$1.129, U$1.25
- removed net OUT3-3.3V: U$1.130, U$1.26
- removed net OUT4-5V: U$1.154, U$1.50
- removed net OUT5-5V: SET_VCC.1, SET_VIN.1, U$1.155, U$1.51
- removed net OUT6-5V: U$1.156, U$1.52
- removed net RX-MAIN: U$1.10, U$1.114
- removed net RX2: U$1.174, U$1.70
- removed net RXD-MAIN: U$1.150, U$1.46
- removed net SPI-CS0: U$1.159, U$1.184, U$1.185, U$1.55, U$1.80, U$1.81
- removed net SPI-MISO: U$1.157, U$1.53
- removed net SPI-MOSI: U$1.183, U$1.79
- removed net SPI-SCK: U$1.158, U$1.54
- removed net TX-MAIN: U$1.140, U$1.36
- removed net TX2: U$1.175, U$1.71
- removed net TXD-MAIN: U$1.124, U$1.20
- removed net VIN: OUT1.2, OUT2.2, OUT3.2, OUT4.2, SET_VIN.2
- removed net V_BAT-VAUX: U$1.101, U$1.179, U$1.205, U$1.75
- new net AIN0: J2.5, U2.PD6(AIN0)
- new net AIN1: J2.6, U2.PD7(AIN1)
- new net ICP: R3.1, U2.PB0(ICP)
- new net INT0: J2.3, U2.PD2(INT0)
- new net INT1: Q1.G, R2.1, U2.PD3(INT1)
- new net OC1A: J2.7, U2.PB1(OC1A)
- new net SCL: I2C.3, U2.PC5(ADC5/SCL)
- new net SDA: I2C.4, U2.PC4(ADC4/SDA)
- new net T0: J2.2, U2.PD4(XCK/T0)
- new net T1: J2.4, U2.PD5(T1)
- net DTR: now also C1.1, FTDI.2; no longer C3.1, JP7.6
- net GND: now also BOOT_LOADER.5, C4.2, C5.2, FTDI.4, I2C.2, J2.11, PAD1.P, Q1.S, R2.2, U2.GND; no longer C1.2, C2.2, ISP6.6, JP7.1, LED13.2, PMV16XNR.S, PMV16XNR1.S, PMV16XNR2.S, PMV16XNR3.S, R11.1, R12.1, R3.2, R4.2, R5.2, R6.2, U$1.171, U$1.197, U$1.198, U$1.67, U$1.93, U$1.94, U1.GND
- net MISO: now also BOOT_LOADER.2, J2.9, U2.PB4(MISO); no longer ISP6.1, U1.PB4(MISO)
- net MOSI: now also BOOT_LOADER.1, J2.8, U2.PB3(MOSI/OC2); no longer ISP6.4, U1.PB3(MOSI/OC2)
- net N$1: now also C5.1, U2.PB6(XTAL1/TOSC1); no longer C1.1, U1.PB6(XTAL1/TOSC1)
- net N$18: now also R3.2; no longer OUT1.1, R10.2
- net N$2: now also C4.1, U2.PB7(XTAL2/TOSC2); no longer C2.1, U1.PB7(XTAL2/TOSC2)
- net N$4: now also Q1.D; no longer LED13.1, R2.1
- net N$6: now also U2.PB2(SS/OC1B); no longer PMV16XNR2.G, R5.1, U1.PD5(T1)
- net RST: now also BOOT_LOADER.4, C1.2, PAD2.P, PAD3.P, R1.2, U2.PC6(/RESET); no longer C3.2, ISP6.5, R1.1, U1.PC6(/RESET)
- net RXD: now also FTDI.5, PAD6.P, PAD7.P, U2.PD0(RXD); no longer JP7.4, R12.2, U1.PD0(RXD)
- net SCK: now also BOOT_LOADER.3, J2.10, U2.PB5(SCK); no longer ISP6.3, R2.2, U1.PB5(SCK)
- net TXD: now also FTDI.6, PAD4.P, PAD5.P, U2.PD1(TXD); no longer JP7.5, R11.2, U1.PD1(TXD)
- net VCC: now also BOOT_LOADER.6, FTDI.3, I2C.1, J2.12, R1.1, U2.AREF, U2.AVCC, U2.VCC; no longer ISP6.2, JP7.3, R1.2, SET_VCC.2, U1.AREF, U1.AVCC, U1.VCC
