File: Electronic/Placa PCB/interstage_A1v2.brd (EAGLE design)
At the start: 82.5 x 29 mm, 18 parts, among them J1 431151015826, Q1 PMV16XNR, T1 MCP9808T-E/MS, T2 MCP9808T-E/MS, U2 ATMEGA328P_TQFP, Y2 ABM3-16.000MHZ-D2Y-T

Commit message: Avance
Parts:
- removed B2/OBC: 53261-7006, SamacSys_Parts:532617006
- removed R_MOS: ERA-8AEB331V, resistor_330_smd:RESC3216X70N
- removed R_PULL1, R_PULL2: ERA-8AEB472V, resistor_4700_smd:RESC3216X70N
- removed R_RST: ERA-8AEB103V, resistor_10000_smd:RESC3216X70N
- added R1: 330, resistor_330_smd:RESC3216X70N
- added R3: 10k, resistor_10000_smd:RESC3216X70N
- added R4, R5: 4.7k, resistor_4700_smd:RESC3216X70N
- added RST: 431151015826, SamacSys_Parts:431151015826
- J1: value 431151015826 -> 53261-7006; device SamacSys_Parts:431151015826 -> SamacSys_Parts:532617006
- R2: value ERA-8AEB331V -> 330
- moved J1 57.7 mm to (9.50, 14.5), turned to 90 degrees
- renumbered BOOTLOADER/FTDI to J4, C4 to C3, C5 to C2, CONEXION_B1 to J2, PINES_SWITCH to J3, Q1 to M1, R_SWITCH to R2, U2 to IC, Y2 to Y1
Connections:
- net GND: now also J1.4, R1.2, RST.3, RST.5, RST.6; no longer B2/OBC.4, J1.3, J1.5, J1.6, R_MOS.2
- net INT1: now also R1.1; no longer R_MOS.1
- net RST: now also R3.1, RST.2; no longer J1.2, R_RST.1
- net SCL: now also J1.1, J1.5, R4.1; no longer B2/OBC.1, B2/OBC.5, R_PULL1.1
- net SDA: now also J1.2, J1.6, R5.1; no longer B2/OBC.2, B2/OBC.6, R_PULL2.1
- net VCC: now also J1.3, R3.2, R4.2, R5.2; no longer B2/OBC.3, R_PULL1.2, R_PULL2.2, R_RST.2
Routing:
- net SCL: track 163.4 -> 162.9 mm
