File: Electronic/Placa PCB/interstage_A1v2.sch (EAGLE design)
At the start: 18 parts, among them J1 431151015826, Q1 PMV16XNR, T1 MCP9808T-E/MS, T2 MCP9808T-E/MS, U2 ATMEGA328P_TQFP, Y2 ABM3-16.000MHZ-D2Y-T

Commit message: Avance
Parts:
- removed B2/OBC: 53261-7006, SamacSys_Parts:53261-7006
- removed BOOTLOADER/FTDI: 53261-1271, SamacSys_Parts:53261-1271
- removed C4, C5: 22pF, rcl:C-EUC0603K
- removed CONEXION_B1: 53261-0871, SamacSys_Parts:53261-0871
- removed R_MOS: ERA-8AEB331V, resistor_330_smd:ERA-8AEB331V
- removed R_PULL1, R_PULL2: ERA-8AEB472V, resistor_4700_smd:ERA-8AEB472V
- removed R_RST: ERA-8AEB103V, resistor_10000_smd:ERA-8AEB103V
- added C2, C3: 22pF, rcl:C-EUC0603K
- added J2: 53261-0871, SamacSys_Parts:53261-0871
- added J4: 53261-1271, SamacSys_Parts:53261-1271
- added R1: 330, resistor_330_smd:ERA-8AEB331V
- added R3: 10k, resistor_10000_smd:ERA-8AEB103V
- added R4, R5: 4.7k, resistor_4700_smd:ERA-8AEB472V
- added RST: 431151015826, SamacSys_Parts:431151015826
- J1: value 431151015826 -> 53261-7006; device SamacSys_Parts:431151015826 -> SamacSys_Parts:53261-7006
- R2: value ERA-8AEB331V -> 330
- renumbered PINES_SWITCH to J3, Q1 to M1, R_SWITCH to R2, U2 to IC, Y2 to Y1
Connections:
- net AIN0: now also J2.4; no longer CONEXION_B1.4
- net AIN1: now also J2.5; no longer CONEXION_B1.5
- net DTR: now also J4.8; no longer BOOTLOADER/FTDI.8
- net GND: now also C2.2, C3.2, J1.4, J2.7, J4.10, J4.5, R1.2, RST.COM_2, RST.GND_1, RST.GND_2; no longer B2/OBC.4, BOOTLOADER/FTDI.10, BOOTLOADER/FTDI.5, C4.2, C5.2, CONEXION_B1.7, J1.COM_2, J1.GND_1, J1.GND_2, R_MOS.2
- net INT0: now also J2.2; no longer CONEXION_B1.2
- net INT1: now also R1.1; no longer R_MOS.1
- net MISO: now also J4.2; no longer BOOTLOADER/FTDI.2
- net MOSI: now also J4.1; no longer BOOTLOADER/FTDI.1
- net N$1: now also C2.1; no longer C5.1
- net N$2: now also C3.1; no longer C4.1
- net OC1A: now also J2.6; no longer CONEXION_B1.6
- net RST: now also J4.4, R3.1, RST.NO_1; no longer BOOTLOADER/FTDI.4, J1.NO_1, R_RST.1
- net RXD: now also J4.11; no longer BOOTLOADER/FTDI.11
- net SCK: now also J4.3; no longer BOOTLOADER/FTDI.3
- net SCL: now also J1.1, J1.5, R4.1; no longer B2/OBC.1, B2/OBC.5, R_PULL1.1
- net SDA: now also J1.2, J1.6, R5.1; no longer B2/OBC.2, B2/OBC.6, R_PULL2.1
- net T0: now also J2.1; no longer CONEXION_B1.1
- net T1: now also J2.3; no longer CONEXION_B1.3
- net TXD: now also J4.12; no longer BOOTLOADER/FTDI.12
- net VCC: now also J1.3, J2.8, J4.6, J4.9, R3.2, R4.2, R5.2; no longer B2/OBC.3, BOOTLOADER/FTDI.6, BOOTLOADER/FTDI.9, CONEXION_B1.8, R_PULL1.2, R_PULL2.2, R_RST.2
Other:
- moved on the sheet: C1, T1, T2
