File: Electronic/Placa PCB/interstage_A2v2.brd (EAGLE design)
At the start: 82.5 x 29 mm, 8 parts, among them Q1 PMV16XNR, T3 MCP9808T-E/MS, T4 MCP9808T-E/MS

Commit message: Avance
Parts:
- removed CONEXION_A1, CONEXION_A2: 53261-0871, SamacSys_Parts:53261-0871
- removed Q1: PMV16XNR, SamacSys_Parts:SOT95P230X110-3N
- removed SV1: (no value), con-lstb:MA03-1
- removed T3, T4: MCP9808T-E/MS, sensorSPEL:SOP65P490X110-8N
- added CONEXION_B1: 53261-0871, SamacSys_Parts:53261-0871
- added CONEXION_B2: 53261-7006, SamacSys_Parts:532617006
- added MOSFET3: PMV16XNR, SamacSys_Parts:SOT95P230X110-3N
- added PINES_SWITCH: (no value), con-lstb:MA03-1
- added T5, T6: MCP9808T-E/MS, sensorSPEL:SOP65P490X110-8N
- moved R_MOSFET 5.50 mm to (29.0, 11.0), turned to 180 degrees
- moved R_SWITCH 3.91 mm to (29.0, 8.00), turned to 180 degrees
Connections:
- removed net AIN1: CONEXION_A1.4, R_SWITCH.2, SV1.2
- removed net T1: CONEXION_A1.6, Q1.1, R_MOSFET.1
- net AIN0: now also CONEXION_B1.6, MOSFET3.1, R_MOSFET.1; no longer CONEXION_A1.5, CONEXION_A2.3
- net GND: now also CONEXION_B1.2, CONEXION_B2.5, MOSFET3.2, T5.4, T5.6, T5.7, T6.4, T6.6; no longer CONEXION_A1.2, CONEXION_A2.7, Q1.2, T3.4, T3.5, T3.7, T4.4, T4.5
- net INT0: now also CONEXION_B1.7, CONEXION_B2.2; no longer CONEXION_A1.7, CONEXION_A2.2
- net NICROMO: now also MOSFET3.3; no longer Q1.3
- net OC1A: now also CONEXION_B1.5, CONEXION_B2.1; no longer CONEXION_A1.3, CONEXION_A2.4
- net SCL: now also CONEXION_B1.3, CONEXION_B2.4, T5.2, T6.2; no longer CONEXION_A2.6, T3.2, T4.2
- net SDA: now also CONEXION_B1.4, CONEXION_B2.3, T5.1, T6.1; no longer CONEXION_A2.5, T3.1, T4.1
- net T0: now also CONEXION_B1.8, PINES_SWITCH.2, R_SWITCH.2; no longer CONEXION_A1.8, CONEXION_A2.1
- net VCC: now also CONEXION_B1.1, CONEXION_B2.6, PINES_SWITCH.1, T5.5, T5.8, T6.5, T6.7, T6.8; no longer CONEXION_A1.1, CONEXION_A2.8, SV1.1, T3.6, T3.8, T4.6, T4.7, T4.8
Routing:
- net SCL: track 53.9 -> 155.2 mm
- net SDA: track 63.9 -> 119.0 mm, vias 1 -> 2
- net T1: track 44.9 -> 0.00 mm
- net INT0: track 46.5 -> 81.6 mm
- net AIN1: track 29.8 -> 0.00 mm, vias 1 -> 0
- net T0: track 46.9 -> 24.5 mm
- net AIN0: track 73.3 -> 58.9 mm, vias 2 -> 0
- net VCC: track 118.1 -> 132.0 mm
- net OC1A: track 83.0 -> 93.9 mm, vias 0 -> 2
- net GND: track 5.75 -> 7.72 mm, vias 1 -> 2
Other:
- outline, holes or cut-outs redrawn

Commit message: Avance
Parts:
- R1, R2: value ERA-8AEB331V -> 330
- renumbered CONEXION_B1 to J1, CONEXION_B2 to J2, MOSFET3 to M1, PINES_SWITCH to J3, R_MOSFET to R1, R_SWITCH to R2, T5 to T1, T6 to T2
Routing:
- net AIN0: track 58.9 -> 61.0 mm
