File: Electronic/Placa PCB/interstage_A2v2.sch (EAGLE design)
At the start: 8 parts, among them Q1 PMV16XNR, T7 MCP9808T-E/MS, T8 MCP9808T-E/MS

Commit message: Avance
Parts:
- removed CONEXION_A1: 0532610271, picoblade2:0532610271
- removed CONEXION_A2: 53261-7006, SamacSys_Parts:53261-7006
- removed Q1: PMV16XNR, SamacSys_Parts:PMV16XNR
- removed SV1: (no value), con-lstb:MA03-1
- removed T7, T8: MCP9808T-E/MS, sensorSPEL:MCP9808T-E/MS
- added CONEXION_B1: 53261-0871, SamacSys_Parts:53261-0871
- added CONEXION_B2: 53261-7006, SamacSys_Parts:53261-7006
- added MOSFET3: PMV16XNR, SamacSys_Parts:PMV16XNR
- added PINES_SWITCH: (no value), con-lstb:MA03-1
- added T5, T6: MCP9808T-E/MS, sensorSPEL:MCP9808T-E/MS
Connections:
- new net AIN0: CONEXION_B1.6, MOSFET3.G, R_MOSFET.1
- new net T0: CONEXION_B1.8, PINES_SWITCH.2, R_SWITCH.2
- net GND: now also CONEXION_B1.2, CONEXION_B2.5, MOSFET3.S, T5.A0, T5.A1, T5.GND, T6.A1, T6.GND; no longer CONEXION_A2.2, Q1.S, T7.A0, T7.GND, T8.GND
- net INT0: now also CONEXION_B1.7, CONEXION_B2.2; no longer CONEXION_A2.6, R_SWITCH.2, SV1.2
- net NICROMO: now also MOSFET3.D; no longer Q1.D
- net OC1A: now also CONEXION_B1.5, CONEXION_B2.1; no longer CONEXION_A2.5, Q1.G, R_MOSFET.1
- net SCL: now also CONEXION_B1.3, CONEXION_B2.4, T5.SCL, T6.SCL; no longer CONEXION_A1.1, CONEXION_A2.3, T7.SCL, T8.SCL
- net SDA: now also CONEXION_B1.4, CONEXION_B2.3, T5.SDA, T6.SDA; no longer CONEXION_A1.2, CONEXION_A2.4, T7.SDA, T8.SDA
- net VCC: now also CONEXION_B1.1, CONEXION_B2.6, PINES_SWITCH.1, T5.A2, T5.VDD, T6.A0, T6.A2, T6.VDD; no longer CONEXION_A2.1, SV1.1, T7.A1, T7.A2, T7.VDD, T8.A0, T8.A1, T8.A2, T8.VDD
Other:
- moved on the sheet: R_MOSFET, R_SWITCH

Commit message: Avance
Parts:
- R1, R2: value ERA-8AEB331V -> 330
- renumbered CONEXION_B1 to J1, CONEXION_B2 to J2, MOSFET3 to M1, PINES_SWITCH to J3, R_MOSFET to R1, R_SWITCH to R2, T5 to T1, T6 to T2
