File: Electronic/Placa PCB/interstage_B1v2.brd (EAGLE design)
At the start: 82.5 x 29 mm, 8 parts, among them Q1 PMV16XNR, T5 MCP9808T-E/MS, T6 MCP9808T-E/MS

Commit message: Avance
Parts:
- removed CONEXION_B1: 53261-0871, SamacSys_Parts:53261-0871
- removed CONEXION_B2: 53261-7006, SamacSys_Parts:532617006
- removed Q1: PMV16XNR, SamacSys_Parts:SOT95P230X110-3N
- removed T5, T6: MCP9808T-E/MS, sensorSPEL:SOP65P490X110-8N
- added CONEXION_A1, CONEXION_A2: 53261-0871, SamacSys_Parts:53261-0871
- added MOSFET2: PMV16XNR, SamacSys_Parts:SOT95P230X110-3N
- added T3, T4: MCP9808T-E/MS, sensorSPEL:SOP65P490X110-8N
- moved PINES_SWITCH 19.8 mm to (4.35, 14.5)
- moved R_MOSFET 5.50 mm to (34.5, 11.0), turned to 90 degrees
- moved R_SWITCH 3.91 mm to (31.5, 11.0), turned to 270 degrees
Connections:
- removed net N$7: PINES_SWITCH.3
- new net AIN1: CONEXION_A1.4, PINES_SWITCH.2, R_SWITCH.2
- new net T1: CONEXION_A1.6, MOSFET2.1, R_MOSFET.1
- net AIN0: now also CONEXION_A1.5, CONEXION_A2.3; no longer CONEXION_B1.6, Q1.1, R_MOSFET.1
- net GND: now also CONEXION_A1.2, CONEXION_A2.7, MOSFET2.2, T3.4, T3.5, T3.7, T4.4, T4.5; no longer CONEXION_B1.2, CONEXION_B2.5, Q1.2, T5.4, T5.6, T5.7, T6.4, T6.6
- net INT0: now also CONEXION_A1.7, CONEXION_A2.2; no longer CONEXION_B1.7, CONEXION_B2.2
- net NICROMO: now also MOSFET2.3; no longer Q1.3
- net OC1A: now also CONEXION_A1.3, CONEXION_A2.4; no longer CONEXION_B1.5, CONEXION_B2.1
- net SCL: now also CONEXION_A2.6, T3.2, T4.2; no longer CONEXION_B1.3, CONEXION_B2.4, T5.2, T6.2
- net SDA: now also CONEXION_A2.5, T3.1, T4.1; no longer CONEXION_B1.4, CONEXION_B2.3, T5.1, T6.1
- net T0: now also CONEXION_A1.8, CONEXION_A2.1; no longer CONEXION_B1.8, PINES_SWITCH.2, R_SWITCH.2
- net VCC: now also CONEXION_A1.1, CONEXION_A2.8, T3.6, T3.8, T4.6, T4.7, T4.8; no longer CONEXION_B1.1, CONEXION_B2.6, T5.5, T5.8, T6.5, T6.7, T6.8
Routing:
- net SCL: track 154.5 -> 53.9 mm
- net SDA: track 119.6 -> 62.7 mm, vias 2 -> 1
- net T1: track 0.00 -> 44.9 mm
- net INT0: track 82.9 -> 46.5 mm
- net AIN1: track 0.00 -> 29.8 mm, vias 0 -> 1
- net T0: track 24.5 -> 46.9 mm
- net AIN0: track 58.9 -> 73.3 mm, vias 0 -> 2
- net VCC: track 131.5 -> 118.1 mm
- net OC1A: track 95.5 -> 83.0 mm, vias 2 -> 0
- net GND: track 7.72 -> 5.75 mm
Other:
- outline, holes or cut-outs redrawn

Commit message: Avance
Parts:
- R1, R2: value ERA-8AEB331V -> 330
- renumbered CONEXION_A1 to J1, CONEXION_A2 to J2, MOSFET2 to M1, PINES_SWITCH to J3, R_MOSFET to R1, R_SWITCH to R2, T3 to T1, T4 to T2
