File: Electronic/Placa PCB/interstage_B2v2.brd (EAGLE design)
At the start: 82.5 x 29 mm, 8 parts, among them Q1 PMV16XNR, T7 MCP9808T-E/MS, T8 MCP9808T-E/MS

Commit message: Avance
Parts:
- renumbered Q1 to MOSFET4, SV1 to PINES_SWITCH
Routing:
- net SCL: track 98.2 -> 97.2 mm
- net OC1A: track 28.4 -> 28.9 mm
Changed lines of the file:
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@@
 </autorouter>
 <elements>
-<element name="Q1" library="SamacSys_Parts" package="SOT95P230X110-3N" value="PMV16XNR" x="34.8" y="14.5" smashed="yes">
+<element name="MOSFET4" library="SamacSys_Parts" package="SOT95P230X110-3N" value="PMV16XNR" x="34.8" y="14.5" smashed="yes">
 <attribute name="DESCRIPTION" value="Nexperia PMV16XNR N-channel MOSFET, 8.6 A, 20 V PMV16XN, 3-Pin SOT-23" x="33.3" y="14.5" size="1.778" layer="27" display="off"/>
 <attribute name="HEIGHT" value="1.1mm" x="33.3" y="14.5" size="1.778" layer="27" display="off"/>
@@
 <attribute name="VALUE" x="25.22695" y="16.94341875" size="1.272740625" layer="27"/>
 </element>
-<element name="SV1" library="con-lstb" library_urn="urn:adsk.eagle:library:162" package="MA03-1" package3d_urn="urn:adsk.eagle:package:8339/1" value="" x="4.35" y="14.5" smashed="yes" rot="R90">
+<element name="PINES_SWITCH" library="con-lstb" library_urn="urn:adsk.eagle:library:162" package="MA03-1" package3d_urn="urn:adsk.eagle:package:8339/1" value="" x="4.35" y="14.5" smashed="yes" rot="R90">
 <attribute name="MF" value="" x="4.35" y="14.5" size="1.778" layer="27" rot="R90" display="off"/>
 <attribute name="MPN" value="" x="4.35" y="14.5" size="1.778" layer="27" rot="R90" display="off"/>
@@
 <signals>
 <signal name="GND">
-<contactref element="Q1" pad="2"/>
+<contactref element="MOSFET4" pad="2"/>
 <contactref element="T7" pad="4"/>
 <contactref element="T8" pad="4"/>
@@
 </signal>
 <signal name="INT0">
-<contactref element="SV1" pad="2"/>
+<contactref element="PINES_SWITCH" pad="2"/>
 <contactref element="CONEXION_A2" pad="6"/>
 <contactref element="R_SWITCH" pad="2"/>
-<wire x1="11.9" y1="11.375" x2="9" y2="11.375" width="0.8" layer="1"/>
-<wire x1="9" y1="11.375" x2="5.875" y2="14.5" width="0.8" layer="1"/>
-<wire x1="5.875" y1="14.5" x2="4.35" y2="14.5" width="0.5" layer="1"/>
+<wire x1="11.9" y1="11.375" x2="8.5" y2="11.375" width="0.8" layer="1"/>
+<wire x1="8.5" y1="11.375" x2="5.375" y2="14.5" width="0.8" layer="1"/>
+<wire x1="5.375" y1="14.5" x2="4.35" y2="14.5" width="0.8" layer="1"/>
 <wire x1="11.9" y1="11.375" x2="14" y2="11.375" width="0.8" layer="1"/>
 <wire x1="14" y1="11.375" x2="19.375" y2="6" width="0.8" layer="1"/>
@@
 </signal>
 <signal name="OC1A">
-<contactref element="Q1" pad="1"/>
+<contactref element="MOSFET4" pad="1"/>
 <contactref element="R_MOSFET" pad="1"/>
 <contactref element="CONEXION_A2" pad="5"/>
 <wire x1="11.9" y1="12.625" x2="16" y2="12.625" width="0.8" layer="1"/>
-<wire x1="30.5" y1="13" x2="30.5" y2="9.025" width="1.5" layer="1"/>
+<wire x1="30.5" y1="14" x2="30.5" y2="9.025" width="1.5" layer="1"/>
 <wire x1="30.525" y1="9" x2="30.5" y2="9.025" width="0.5" layer="1"/>
-<wire x1="33.7" y1="15.45" x2="32.95" y2="15.45" width="1.5" layer="1"/>
-<wire x1="32.95" y1="15.45" x2="30.5" y2="13" width="1.5" layer="1"/>
+<wire x1="33.7" y1="15.45" x2="31.95" y2="15.45" width="1.5" layer="1"/>
+<wire x1="31.95" y1="15.45" x2="30.5" y2="14" width="1.5" layer="1"/>
 <wire x1="16" y1="12.625" x2="19.625" y2="9" width="1.5" layer="1"/>
-<wire x1="19.625" y1="9" x2="26.5" y2="9" width="1.5" layer="1"/>
-<wire x1="26.5" y1="9" x2="30.525" y2="9" width="1.5" layer="1"/>
+<wire x1="19.625" y1="9" x2="30.525" y2="9" width="1.5" layer="1"/>
 </signal>
 <signal name="NICROMO">
-<contactref element="Q1" pad="3"/>
+<contactref element="MOSFET4" pad="3"/>
 <via x="40" y="14.5" extent="1-16" drill="1.8" diameter="4"/>
 <wire x1="35.9" y1="14.5" x2="40" y2="14.5" width="1.5" layer="1"/>
@@
 <contactref element="T8" pad="6"/>
 <wire x1="19.8" y1="19.025" x2="17.475" y2="19.025" width="0.5" layer="16"/>
-<contactref element="SV1" pad="1"/>
+<contactref element="PINES_SWITCH" pad="1"/>
 <contactref element="CONEXION_A2" pad="1"/>
 <wire x1="11.9" y1="17.625" x2="14.275" y2="17.625" width="0.8" layer="1"/>
@@
 <wire x1="24.2" y1="20.325" x2="27" y2="20.325" width="0.5" layer="16"/>
 <wire x1="45.2" y1="20.325" x2="44" y2="20.325" width="0.5" layer="16"/>
-<wire x1="45.2" y1="20.325" x2="47.5" y2="20.325" width="0.5" layer="16"/>
+<wire x1="45.2" y1="20.325" x2="46.5" y2="20.325" width="0.5" layer="16"/>
 <via x="46" y="6.5" extent="1-16" drill="0.35" diameter="1"/>
-<wire x1="48" y1="19.825" x2="47.5" y2="20.325" width="0.5" layer="16"/>
-<wire x1="48" y1="19.825" x2="48" y2="8.5" width="0.8" layer="16"/>
+<wire x1="47.5" y1="19.325" x2="46.5" y2="20.325" width="0.5" layer="16"/>
+<wire x1="47.5" y1="19.325" x2="47.5" y2="8" width="0.8" layer="16"/>
 <wire x1="46" y1="6.625" x2="42.5" y2="6.625" width="0.8" layer="1"/>
 <wire x1="46" y1="6.625" x2="46" y2="6.5" width="0.8" layer="1"/>
@@
 <wire x1="27" y1="20.325" x2="27.7" y2="21.025" width="0.5" layer="16"/>
 <wire x1="27.7" y1="21.025" x2="27.7" y2="24.5" width="0.5" layer="16"/>
-<wire x1="46" y1="6.5" x2="48" y2="8.5" width="0.8" layer="16"/>
+<wire x1="46" y1="6.5" x2="47.5" y2="8" width="0.8" layer="16"/>
 </signal>
 <signal name="SDA">
@@
 <contactref element="CONEXION_A2" pad="4"/>
 <via x="7.5" y="15.5" extent="1-16" drill="0.35" diameter="1"/>
-<wire x1="48" y1="24.5" x2="48" y2="23" width="0.8" layer="16"/>
 <wire x1="45.2" y1="20.975" x2="46.5" y2="20.975" width="0.5" layer="16"/>
 <wire x1="26.4" y1="21.875" x2="26.4" y2="27" width="0.5" layer="16"/>
@@
 <wire x1="36.5" y1="2" x2="10.5" y2="2" width="0.8" layer="1"/>
 <via x="10.5" y="2" extent="1-16" drill="0.35" diameter="1"/>
-<wire x1="11.9" y1="13.875" x2="9.125" y2="13.875" width="0.8" layer="1"/>
-<wire x1="9.125" y1="13.875" x2="7.5" y2="15.5" width="0.8" layer="1"/>
+<wire x1="11.9" y1="13.875" x2="8.625" y2="13.875" width="0.8" layer="1"/>
+<wire x1="8.625" y1="13.875" x2="7.5" y2="15" width="0.8" layer="1"/>
+<wire x1="7.5" y1="15" x2="7.5" y2="15.5" width="0.8" layer="1"/>
 <wire x1="10.5" y1="2" x2="9" y2="2" width="0.8" layer="16"/>
 <wire x1="9" y1="2" x2="7.5" y2="3.5" width="0.8" layer="16"/>
@@
 <wire x1="7.5" y1="24" x2="10.5" y2="27" width="0.8" layer="16"/>
 <wire x1="10.5" y1="27" x2="26.4" y2="27" width="0.8" layer="16"/>
-<wire x1="45.5" y1="27" x2="48" y2="24.5" width="0.8" layer="16"/>
-<wire x1="46.5" y1="20.975" x2="48" y2="22.475" width="0.5" layer="16"/>
-<wire x1="48" y1="22.475" x2="48" y2="23" width="0.5" layer="16"/>
+<wire x1="45.5" y1="27" x2="47.5" y2="25" width="0.8" layer="16"/>
+<wire x1="47.5" y1="21.975" x2="46.5" y2="20.975" width="0.5" layer="16"/>
 <wire x1="25.5" y1="20.975" x2="26.4" y2="21.875" width="0.5" layer="16"/>
+<wire x1="47.5" y1="25" x2="47.5" y2="21.975" width="0.8" layer="16"/>
 </signal>
 </signals>
@@
 <mfgpreviewcolor name="substratecolor" color="0xFF786E46"/>
 </mfgpreviewcolors>
+<errors>
+</errors>
 </board>
 </drawing>

Commit message: Avance
Parts:
- removed CONEXION_A1: 0532610271, picoblade2:MOLEX_0532610271
- removed CONEXION_A2: 53261-7006, SamacSys_Parts:532617006
- removed R_MOSFET, R_SWITCH: ERA-8AEB331V, resistor_330_smd:RESC3216X70N
- removed T7, T8: MCP9808T-E/MS, sensorSPEL:SOP65P490X110-8N
- added J1: 53261-7006, SamacSys_Parts:532617006
- added J2: 0532610271, picoblade2:MOLEX_0532610271
- added R1, R2: 330, resistor_330_smd:RESC3216X70N
- added T1, T2: MCP9808T-E/MS, sensorSPEL:SOP65P490X110-8N
- renumbered MOSFET4 to M1, PINES_SWITCH to J3
Connections:
- net GND: now also J1.2, R1.2, R2.1, T1.4, T1.7, T2.4; no longer CONEXION_A2.2, R_MOSFET.2, R_SWITCH.1, T7.4, T7.7, T8.4
- net INT0: now also J1.6, R2.2; no longer CONEXION_A2.6, R_SWITCH.2
- net OC1A: now also J1.5, R1.1; no longer CONEXION_A2.5, R_MOSFET.1
- net SCL: now also J1.3, J2.1, T1.2, T2.2; no longer CONEXION_A1.1, CONEXION_A2.3, T7.2, T8.2
- net SDA: now also J1.4, J2.2, T1.1, T2.1; no longer CONEXION_A1.2, CONEXION_A2.4, T7.1, T8.1
- net VCC: now also J1.1, T1.5, T1.6, T1.8, T2.5, T2.6, T2.7, T2.8; no longer CONEXION_A2.1, T7.5, T7.6, T7.8, T8.5, T8.6, T8.7, T8.8
Routing:
- net SDA: track 118.4 -> 102.9 mm
- net SCL: track 97.2 -> 83.6 mm
- net OC1A: track 28.9 -> 22.9 mm
- net VCC: track 87.6 -> 82.5 mm
- net INT0: track 29.7 -> 27.3 mm
