File: Electronic/Placa PCB/interstage_B2v2.sch (EAGLE design)
At the start: 8 parts, among them Q1 PMV16XNR, T3 MCP9808T-E/MS, T4 MCP9808T-E/MS

Commit message: Avance
Parts:
- removed Q1: PMV16XNR, SamacSys_Parts:PMV16XNR
- removed SV1: (no value), con-lstb:MA03-1
- removed T3, T4: MCP9808T-E/MS, sensorSPEL:MCP9808T-E/MS
- added MOSFET4: PMV16XNR, SamacSys_Parts:PMV16XNR
- added PINES_SWITCH: (no value), con-lstb:MA03-1
- added T7, T8: MCP9808T-E/MS, sensorSPEL:MCP9808T-E/MS
- CONEXION_A1: value 53261-0871 -> 0532610271; device SamacSys_Parts:53261-0871 -> picoblade2:0532610271
- CONEXION_A2: value 53261-0871 -> 53261-7006; device SamacSys_Parts:53261-0871 -> SamacSys_Parts:53261-7006
Connections:
- removed net AIN0: CONEXION_A1.5, CONEXION_A2.3
- removed net AIN1: CONEXION_A1.4, R_SWITCH.2, SV1.2
- removed net T0: CONEXION_A1.8, CONEXION_A2.1
- removed net T1: CONEXION_A1.6, Q1.G, R_MOSFET.1
- net GND: now also CONEXION_A2.2, MOSFET4.S, T7.A0, T7.GND, T8.GND; no longer CONEXION_A1.2, CONEXION_A2.7, Q1.S, T3.A0, T3.A2, T3.GND, T4.A2, T4.GND
- net INT0: now also CONEXION_A2.6, PINES_SWITCH.2, R_SWITCH.2; no longer CONEXION_A1.7, CONEXION_A2.2
- net NICROMO: now also MOSFET4.D; no longer Q1.D
- net OC1A: now also CONEXION_A2.5, MOSFET4.G, R_MOSFET.1; no longer CONEXION_A1.3, CONEXION_A2.4
- net SCL: now also CONEXION_A1.1, CONEXION_A2.3, T7.SCL, T8.SCL; no longer CONEXION_A2.6, T3.SCL, T4.SCL
- net SDA: now also CONEXION_A1.2, CONEXION_A2.4, T7.SDA, T8.SDA; no longer CONEXION_A2.5, T3.SDA, T4.SDA
- net VCC: now also CONEXION_A2.1, PINES_SWITCH.1, T7.A1, T7.A2, T7.VDD, T8.A0, T8.A1, T8.A2, T8.VDD; no longer CONEXION_A1.1, CONEXION_A2.8, SV1.1, T3.A1, T3.VDD, T4.A0, T4.A1, T4.VDD
Other:
- moved on the sheet: CONEXION_A2, R_MOSFET, R_SWITCH

Commit message: Avance
Parts:
- R1, R2: value ERA-8AEB331V -> 330
- renumbered CONEXION_A1 to J2, CONEXION_A2 to J1, MOSFET4 to M1, PINES_SWITCH to J3, R_MOSFET to R1, R_SWITCH to R2, T7 to T1, T8 to T2
