File: Electronic/Placa PCB/v1/interstage_A1.sch (EAGLE design)
At the start: 11 parts, among them J1 0532611271, J3 0532611271, Q1 PMV16XNR, U1 LM70CIMM-3, U2 LM70CIMM-3

Commit message: Avance
Parts:
- removed C2: 0.1pF, rcl:C-EUC0603K
- removed J3: 0532611271, picoblade:0532611271
- removed PAD1, PAD2: WIREPADSMD1,27-254, wirepad:WIREPADSMD1,27-254
- removed R5, R9: 330 Ohm, rcl:R-EU_R1206
- removed U1: LM70CIMM-3, LM70CIMM-3:LM70CIMM-3
- added BOOT_LOADER, FTDI: 0532610671, picoblade6:0532610671
- added C4, C5: 22pF, rcl:C-EUC0603K
- added I2C: 0532610471, 0532610471:0532610471
- added J2: 0532611271, picoblade:0532611271
- added R1: 10kohm, rcl:R-EU_R1206
- added R2, R3: 330 Ohm, rcl:R-EU_R1206
- added S1: (no value), switch-omron:10-XX
- added Y1: 16MHz, SparkFun-Clocks:CRYSTAL-16MHZSMD-2X1.6
- C1: value 0.1pF -> 100nF; device rcl:C-EUC0603K -> rcl:C-EUC0805K
- U2: value LM70CIMM-3 -> ATMEGA328P_TQFP; device LM70CIMM-3:LM70CIMM-3 -> SparkFun-IC-Microcontroller:ATMEGA328P_TQFP
Connections:
- net MOSFET renamed NICROMO
- removed net N$3: J3.1
- removed net N$4: R9.1
- new net DTR: C1.1, FTDI.2
- new net ICP: R3.1, U2.PB0(ICP)
- new net INT1: Q1.G, R2.1, U2.PD3(INT1)
- new net N$1: C5.1, U2.PB6(XTAL1/TOSC1), Y1.1
- new net N$2: C4.1, U2.PB7(XTAL2/TOSC2), Y1.2
- new net N$6: U2.PB2(SS/OC1B)
- new net RST: BOOT_LOADER.4, C1.2, R1.2, S1.S, S1.S1, U2.PC6(/RESET)
- new net RXD: FTDI.5, U2.PD0(RXD)
- new net SCL: I2C.3, U2.PC5(ADC5/SCL)
- new net SDA: I2C.4, U2.PC4(ADC4/SDA)
- new net SWITCH: R3.2
- new net TXD: FTDI.6, U2.PD1(TXD)
- net AIN0: now also J2.5, U2.PD6(AIN0); no longer J1.8, J3.5
- net AIN1: now also J2.6, U2.PD7(AIN1); no longer J1.7, J3.6, R9.2
- net GND: now also BOOT_LOADER.5, C4.2, C5.2, FTDI.4, I2C.2, J2.11, R2.2, S1.P, S1.P1; no longer C1.2, C2.2, J1.2, J3.11, PAD1.P, PAD2.P, R5.1, U1.GND
- net INT0: now also J2.3, U2.PD2(INT0); no longer J1.10, J3.3
- net MISO: now also BOOT_LOADER.2, J2.9, U2.PB4(MISO); no longer J1.4, J3.9, U1.SI/O, U2.SI/O
- net MOSI: now also BOOT_LOADER.1, J2.8, U2.PB3(MOSI/OC2); no longer J1.5, J3.8, U1.~CS, U2.~CS
- net OC1A: now also J2.7, U2.PB1(OC1A); no longer J1.6, J3.7, Q1.G, R5.2
- net SCK: now also BOOT_LOADER.3, J2.10, U2.PB5(SCK); no longer J1.3, J3.10, U1.SC, U2.SC
- net T0: now also J2.2, U2.PD4(XCK/T0); no longer J1.11, J3.2
- net T1: now also J2.4, U2.PD5(T1); no longer J1.9, J3.4
- net VCC: now also BOOT_LOADER.6, FTDI.3, I2C.1, J2.12, R1.1, U2.AREF, U2.AVCC, U2.VCC; no longer C1.1, C2.1, J1.1, J3.12, U1.V+, U2.V+
Other:
- moved on the sheet: C1, J1, Q1
