File: Electronic/Placa PCB/v1/interstage_B1.sch (EAGLE design)
At the start: 11 parts, among them J1 0532611271, J3 0532611271, Q1 PMV16XNR, U1 LM70CIMM-3, U2 LM70CIMM-3

Commit message: Avance
Parts:
- removed PAD1, PAD2: WIREPADSMD1,27-254, wirepad:WIREPADSMD1,27-254
Connections:
- net GND: no longer PAD1.P, PAD2.P
Changed lines of the file:
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@@
 <?xml version="1.0" encoding="utf-8"?>
 <!DOCTYPE eagle SYSTEM "eagle.dtd">
-<eagle version="9.6.0">
+<eagle version="9.6.1">
 <drawing>
 <settings>
@@
 <part name="Q1" library="SamacSys_Parts" deviceset="PMV16XNR" device=""/>
 <part name="J3" library="picoblade" deviceset="0532611271" device=""/>
-<part name="PAD1" library="wirepad" library_urn="urn:adsk.eagle:library:412" deviceset="WIREPAD" device="SMD1,27-254" package3d_urn="urn:adsk.eagle:package:30839/1"/>
-<part name="PAD2" library="wirepad" library_urn="urn:adsk.eagle:library:412" deviceset="WIREPAD" device="SMD1,27-254" package3d_urn="urn:adsk.eagle:package:30839/1"/>
 <part name="C1" library="rcl" library_urn="urn:adsk.eagle:library:334" deviceset="C-EU" device="C0603K" package3d_urn="urn:adsk.eagle:package:23680/2" value="0.1pF"/>
 <part name="C2" library="rcl" library_urn="urn:adsk.eagle:library:334" deviceset="C-EU" device="C0603K" package3d_urn="urn:adsk.eagle:package:23680/2" value="0.1pF"/>
@@
 <attribute name="NAME" x="245.11" y="27.94" size="1.778" layer="95"/>
 <attribute name="VALUE" x="245.11" y="-12.7" size="1.778" layer="96"/>
-</instance>
-<instance part="PAD1" gate="G$1" x="193.04" y="87.63" smashed="yes" rot="R180">
-<attribute name="NAME" x="194.183" y="85.7758" size="1.778" layer="95" rot="R180"/>
-<attribute name="VALUE" x="194.183" y="90.932" size="1.778" layer="96" rot="R180"/>
-</instance>
-<instance part="PAD2" gate="G$1" x="193.04" y="81.28" smashed="yes" rot="R180">
-<attribute name="NAME" x="194.183" y="79.4258" size="1.778" layer="95" rot="R180"/>
-<attribute name="VALUE" x="194.183" y="84.582" size="1.778" layer="96" rot="R180"/>
 </instance>
 <instance part="C1" gate="G$1" x="85.09" y="113.03" smashed="yes">
@@
 <label x="227.33" y="0" size="1.778" layer="95" rot="R180" xref="yes"/>
 </segment>
-<segment>
-<pinref part="PAD1" gate="G$1" pin="P"/>
-<wire x1="190.5" y1="87.63" x2="187.96" y2="87.63" width="0.1524" layer="91"/>
-<label x="187.96" y="87.63" size="1.778" layer="95" rot="R180" xref="yes"/>
-</segment>
-<segment>
-<pinref part="PAD2" gate="G$1" pin="P"/>
-<wire x1="190.5" y1="81.28" x2="187.96" y2="81.28" width="0.1524" layer="91"/>
-<label x="187.96" y="81.28" size="1.778" layer="95" rot="R180" xref="yes"/>
-</segment>
 </net>
