File: Electronic/Placa PCB/v2/interstage_A1v2.brd (EAGLE design)
At the start: 82.5 x 29 mm, 15 parts, among them Q1 PMV16XNR, U1 MCP9808T-E/MS, U2 ATMEGA328P_TQFP, U3 MCP9808T-E/MS, Y2 ABM3-16.000MHZ-D2Y-T

Commit message: Placas PCB
Parts:
- removed BOOT_LOADER/FTDI: 0532611271, picoblade:MOLEX_0532611271
- removed I2C_PLACAS/I2C_OBC: 53261-0871, SamacSys_Parts:53261-0871
- removed R1: 10kohm, rcl:R1206
- removed R2, R3: 330 Ohm, rcl:R1206
- removed S1: (no value), switch-omron:B3F-10XX
- removed U1, U3: MCP9808T-E/MS, sensorSPEL:SOP65P490X110-8N
- added B2/OBC: 53261-7006, SamacSys_Parts:532617006
- added BOOTLOADER/FTDI: 53261-1271, SamacSys_Parts:53261-1271
- added J1: 431151015826, SamacSys_Parts:431151015826
- added PINES_SWITCH: (no value), con-lstb:MA03-1
- added R_MOS, R_SWITCH: ERA-8AEB331V, resistor_330_smd:RESC3216X70N
- added R_PULL1, R_PULL2: ERA-8AEB472V, resistor_4700_smd:RESC3216X70N
- added R_RST: ERA-8AEB103V, resistor_10000_smd:RESC3216X70N
- added T1, T2: MCP9808T-E/MS, sensorSPEL:SOP65P490X110-8N
- renumbered I2C_PLACAS/I2C_OBC1 to CONEXION_B1
Connections:
- removed net ICP: R3.1, U2.12
- removed net N$6: U2.14
- net DTR: now also BOOTLOADER/FTDI.8; no longer BOOT_LOADER/FTDI.8
- net GND: now also B2/OBC.4, BOOTLOADER/FTDI.10, BOOTLOADER/FTDI.5, J1.3, J1.5, J1.6, R_MOS.2, R_SWITCH.1, T1.4, T1.5, T1.6, T1.7, T2.4, T2.5, T2.6; no longer BOOT_LOADER/FTDI.10, BOOT_LOADER/FTDI.5, I2C_PLACAS/I2C_OBC.2, I2C_PLACAS/I2C_OBC.6, R2.2, S1.3, S1.4, U1.4, U3.4
- net INT1: now also R_MOS.1; no longer R2.1
- net MISO: now also BOOTLOADER/FTDI.2; no longer BOOT_LOADER/FTDI.2
- net MOSI: now also BOOTLOADER/FTDI.1; no longer BOOT_LOADER/FTDI.1
- net RST: now also BOOTLOADER/FTDI.4, J1.2, R_RST.1; no longer BOOT_LOADER/FTDI.4, R1.2, S1.1, S1.2
- net RXD: now also BOOTLOADER/FTDI.11; no longer BOOT_LOADER/FTDI.11
- net SCK: now also BOOTLOADER/FTDI.3; no longer BOOT_LOADER/FTDI.3
- net SCL: now also B2/OBC.1, B2/OBC.5, R_PULL1.1, T1.2, T2.2; no longer I2C_PLACAS/I2C_OBC.3, I2C_PLACAS/I2C_OBC.7, U1.2, U3.2
- net SDA: now also B2/OBC.2, B2/OBC.6, R_PULL2.1, T1.1, T2.1; no longer I2C_PLACAS/I2C_OBC.4, I2C_PLACAS/I2C_OBC.8, U1.1, U3.1
- net SWITCH: now also PINES_SWITCH.2, R_SWITCH.2, U2.12; no longer R3.2
- net TXD: now also BOOTLOADER/FTDI.12; no longer BOOT_LOADER/FTDI.12
- net VCC: now also B2/OBC.3, BOOTLOADER/FTDI.6, BOOTLOADER/FTDI.9, PINES_SWITCH.1, R_PULL1.2, R_PULL2.2, R_RST.2, T1.8, T2.7, T2.8; no longer BOOT_LOADER/FTDI.6, BOOT_LOADER/FTDI.9, I2C_PLACAS/I2C_OBC.1, I2C_PLACAS/I2C_OBC.5, R1.1, U1.8, U3.8
Routing:
- net SWITCH: track 2.08 -> 118.7 mm
- net SCL: track 94.6 -> 161.9 mm, vias 2 -> 3
- net SDA: track 77.7 -> 117.7 mm
- net ICP: track 31.4 -> 0.00 mm
- net VCC: track 188.3 -> 204.9 mm, vias 4 -> 1
- net RST: track 140.8 -> 132.1 mm, vias 3 -> 4
- net RXD: track 102.0 -> 109.4 mm
- net OC1A: track 49.0 -> 55.6 mm, vias 0 -> 2
- net TXD: track 88.2 -> 94.8 mm
- net INT1: track 36.6 -> 33.5 mm
- net INT0: track 55.8 -> 57.9 mm
- net GND: track 0.00 -> 2.03 mm, vias 2 -> 5
- net MISO: track 10.9 -> 8.89 mm
- net MOSI: track 10.4 -> 8.70 mm
- net T1: track 39.4 -> 40.9 mm, vias 0 -> 2
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Other:
- outline, holes or cut-outs redrawn
