File: Electronic/Placa PCB/v2/interstage_A1v2.sch (EAGLE design)
At the start: 15 parts, among them Q1 PMV16XNR, U1 MCP9808T-E/MS, U2 ATMEGA328P_TQFP, U3 MCP9808T-E/MS, Y2 ABM3-16.000MHZ-D2Y-T

Commit message: Placas PCB
Parts:
- removed BOOT_LOADER/FTDI: 0532611271, picoblade:0532611271
- removed I2C_PLACAS/I2C_OBC, I2C_PLACAS/I2C_OBC1: 53261-0871, SamacSys_Parts:53261-0871
- removed R1: 10kohm, rcl:R-EU_R1206
- removed R2, R3: 330 Ohm, rcl:R-EU_R1206
- removed S1: (no value), switch-omron:10-XX
- removed U1, U3: MCP9808T-E/MS, sensorSPEL:MCP9808T-E/MS
- added B2/OBC: 53261-7006, SamacSys_Parts:53261-7006
- added BOOTLOADER/FTDI: 53261-1271, SamacSys_Parts:53261-1271
- added CONEXION_B1: 53261-0871, SamacSys_Parts:53261-0871
- added J1: 431151015826, SamacSys_Parts:431151015826
- added PINES_SWITCH: (no value), con-lstb:MA03-1
- added R_MOS, R_SWITCH: ERA-8AEB331V, resistor_330_smd:ERA-8AEB331V
- added R_PULL1, R_PULL2: ERA-8AEB472V, resistor_4700_smd:ERA-8AEB472V
- added R_RST: ERA-8AEB103V, resistor_10000_smd:ERA-8AEB103V
- added T1, T2: MCP9808T-E/MS, sensorSPEL:MCP9808T-E/MS
Connections:
- removed net ICP: R3.1, U2.PB0(ICP)
- removed net N$6: U2.PB2(SS/OC1B)
- net AIN0: now also CONEXION_B1.4; no longer I2C_PLACAS/I2C_OBC1.4
- net AIN1: now also CONEXION_B1.5; no longer I2C_PLACAS/I2C_OBC1.5
- net DTR: now also BOOTLOADER/FTDI.8; no longer BOOT_LOADER/FTDI.8
- net GND: now also B2/OBC.4, BOOTLOADER/FTDI.10, BOOTLOADER/FTDI.5, CONEXION_B1.7, J1.COM_2, J1.GND_1, J1.GND_2, R_MOS.2, R_SWITCH.1, T1.A0, T1.A1, T1.A2, T1.GND, T2.A1, T2.A2, T2.GND; no longer BOOT_LOADER/FTDI.10, BOOT_LOADER/FTDI.5, I2C_PLACAS/I2C_OBC.2, I2C_PLACAS/I2C_OBC.6, I2C_PLACAS/I2C_OBC1.7, R2.2, S1.P, S1.P1, U1.GND, U3.GND
- net INT0: now also CONEXION_B1.2; no longer I2C_PLACAS/I2C_OBC1.2
- net INT1: now also R_MOS.1; no longer R2.1
- net MISO: now also BOOTLOADER/FTDI.2; no longer BOOT_LOADER/FTDI.2
- net MOSI: now also BOOTLOADER/FTDI.1; no longer BOOT_LOADER/FTDI.1
- net OC1A: now also CONEXION_B1.6; no longer I2C_PLACAS/I2C_OBC1.6
- net RST: now also BOOTLOADER/FTDI.4, J1.NO_1, R_RST.1; no longer BOOT_LOADER/FTDI.4, R1.2, S1.S, S1.S1
- net RXD: now also BOOTLOADER/FTDI.11; no longer BOOT_LOADER/FTDI.11
- net SCK: now also BOOTLOADER/FTDI.3; no longer BOOT_LOADER/FTDI.3
- net SCL: now also B2/OBC.1, B2/OBC.5, R_PULL1.1, T1.SCL, T2.SCL; no longer I2C_PLACAS/I2C_OBC.3, I2C_PLACAS/I2C_OBC.7, U1.SCL, U3.SCL
- net SDA: now also B2/OBC.2, B2/OBC.6, R_PULL2.1, T1.SDA, T2.SDA; no longer I2C_PLACAS/I2C_OBC.4, I2C_PLACAS/I2C_OBC.8, U1.SDA, U3.SDA
- net SWITCH: now also PINES_SWITCH.2, R_SWITCH.2, U2.PB0(ICP); no longer R3.2
- net T0: now also CONEXION_B1.1; no longer I2C_PLACAS/I2C_OBC1.1
- net T1: now also CONEXION_B1.3; no longer I2C_PLACAS/I2C_OBC1.3
- net TXD: now also BOOTLOADER/FTDI.12; no longer BOOT_LOADER/FTDI.12
- net VCC: now also B2/OBC.3, BOOTLOADER/FTDI.6, BOOTLOADER/FTDI.9, CONEXION_B1.8, PINES_SWITCH.1, R_PULL1.2, R_PULL2.2, R_RST.2, T1.VDD, T2.A0, T2.VDD; no longer BOOT_LOADER/FTDI.6, BOOT_LOADER/FTDI.9, I2C_PLACAS/I2C_OBC.1, I2C_PLACAS/I2C_OBC.5, I2C_PLACAS/I2C_OBC1.8, R1.1, U1.VDD, U3.VDD
Other:
- moved on the sheet: Q1
