File: Electronic/Placa PCB/v2/interstage_A2v2.brd (EAGLE design)
At the start: 82.5 x 29 mm, 11 parts, among them J1 0532611271, J3 0532611271, Q1 PMV16XNR, U1 LM70CIMM-3, U2 LM70CIMM-3

Commit message: Avance
Parts:
- removed C1, C2: 0.1pF, rcl:C0603K
- removed J1, J3: 0532611271, picoblade:MOLEX_0532611271
- removed PAD1, PAD2: WIREPADSMD1,27-254, wirepad:SMD1,27-2,54
- removed U2: LM70CIMM-3, LM70CIMM-3:SOP65P490X110-8N
- added I2C_PLACAS/I2C_OBC, I2C_PLACAS/I2C_OBC1: 53261-0871, SamacSys_Parts:53261-0871
- added U3: MCP9808T-E/MS, sensorSPEL:SOP65P490X110-8N
- U1: value LM70CIMM-3 -> MCP9808T-E/MS; device LM70CIMM-3:SOP65P490X110-8N -> sensorSPEL:SOP65P490X110-8N
- moved U1 13.5 mm to (32.5, 20.0)
- moved Q1 8.51 mm to (27.9, 14.5)
- moved R9 7.55 mm to (23.6, 4.40)
- moved R5 3.71 mm to (19.2, 7.70), turned to 90 degrees
Connections:
- removed net AIN1: J1.7, J3.6
- removed net MISO: J1.4, J3.9, U1.1, U2.1
- removed net MOSI: J1.5, J3.8, U1.7, U2.7
- removed net N$3: J3.1
- removed net SCK: J1.3, J3.10, U1.2, U2.2
- removed net T1: J1.9, J3.4, Q1.1, R5.2
- new net SCL: I2C_PLACAS/I2C_OBC.3, I2C_PLACAS/I2C_OBC1.6, U1.2, U3.2
- new net SDA: I2C_PLACAS/I2C_OBC.4, I2C_PLACAS/I2C_OBC1.5, U1.1, U3.1
- net AIN0: now also I2C_PLACAS/I2C_OBC.6, Q1.1, R5.2; no longer J1.8, J3.5
- net GND: now also I2C_PLACAS/I2C_OBC.2, I2C_PLACAS/I2C_OBC1.7, U3.4; no longer C1.2, C2.2, J1.2, J3.11, PAD1.1, PAD2.1, U2.4
- net INT0: now also I2C_PLACAS/I2C_OBC.7, I2C_PLACAS/I2C_OBC1.4; no longer J1.10, J3.3, R9.2
- net OC1A: now also I2C_PLACAS/I2C_OBC.5, I2C_PLACAS/I2C_OBC1.3; no longer J1.6, J3.7
- net T0: now also I2C_PLACAS/I2C_OBC.8, R9.2; no longer J1.11, J3.2
- net VCC: now also I2C_PLACAS/I2C_OBC.1, I2C_PLACAS/I2C_OBC1.8, U1.8, U3.8; no longer C1.1, C2.1, J1.1, J3.12, U1.5, U2.5
Routing:
- net SDA: track 0.00 -> 132.8 mm, vias 0 -> 2
- net MISO: track 129.8 -> 0.00 mm, vias 1 -> 0
- net SCL: track 0.00 -> 124.9 mm, vias 0 -> 2
- net SCK: track 118.1 -> 0.00 mm, vias 1 -> 0
- net T1: track 95.7 -> 0.00 mm
- net MOSI: track 89.1 -> 0.00 mm, vias 1 -> 0
- net AIN1: track 59.3 -> 0.00 mm
- net T0: track 53.8 -> 11.4 mm
- net OC1A: track 58.5 -> 100.8 mm
- net AIN0: track 60.8 -> 22.1 mm
- net GND: track 29.2 -> 0.00 mm
- net INT0: track 55.9 -> 82.7 mm
- net VCC: track 113.2 -> 123.1 mm, vias 1 -> 3
Other:
- outline, holes or cut-outs redrawn

Commit message: Placas PCB
Parts:
- removed I2C_PLACAS/I2C_OBC, I2C_PLACAS/I2C_OBC1: 53261-0871, SamacSys_Parts:53261-0871
- removed R5, R9: 330 Ohm, rcl:R1206
- added CONEXION_B1: 53261-0871, SamacSys_Parts:53261-0871
- added CONEXION_B2: 53261-7006, SamacSys_Parts:532617006
- added PINES_SWITCH: (no value), con-lstb:MA03-1
- added R_MOSFET, R_SWITCH: ERA-8AEB331V, resistor_330_smd:RESC3216X70N
- moved Q1 26.6 mm to (54.5, 14.5), turned to 180 degrees
- renumbered U1 to T5, U3 to T6
Connections:
- net MOSFET renamed NICROMO
- removed net N$4: R9.1
- new net N$7: PINES_SWITCH.3
- net AIN0: now also CONEXION_B1.6, R_MOSFET.1; no longer I2C_PLACAS/I2C_OBC.6, R5.2
- net GND: now also CONEXION_B1.2, CONEXION_B2.5, R_MOSFET.2, R_SWITCH.1, T5.6, T5.7, T6.6; no longer I2C_PLACAS/I2C_OBC.2, I2C_PLACAS/I2C_OBC1.7, R5.1
- net INT0: now also CONEXION_B1.7, CONEXION_B2.2; no longer I2C_PLACAS/I2C_OBC.7, I2C_PLACAS/I2C_OBC1.4
- net OC1A: now also CONEXION_B1.5, CONEXION_B2.1; no longer I2C_PLACAS/I2C_OBC.5, I2C_PLACAS/I2C_OBC1.3
- net SCL: now also CONEXION_B1.3, CONEXION_B2.4; no longer I2C_PLACAS/I2C_OBC.3, I2C_PLACAS/I2C_OBC1.6
- net SDA: now also CONEXION_B1.4, CONEXION_B2.3; no longer I2C_PLACAS/I2C_OBC.4, I2C_PLACAS/I2C_OBC1.5
- net T0: now also CONEXION_B1.8, PINES_SWITCH.2, R_SWITCH.2; no longer I2C_PLACAS/I2C_OBC.8, R9.2
- net VCC: now also CONEXION_B1.1, CONEXION_B2.6, PINES_SWITCH.1, T5.5, T6.5, T6.7; no longer I2C_PLACAS/I2C_OBC.1, I2C_PLACAS/I2C_OBC1.8
Routing:
- net AIN0: track 22.1 -> 72.4 mm, vias 0 -> 2
- net SCL: track 124.9 -> 170.7 mm, vias 2 -> 1
- net T0: track 11.4 -> 25.2 mm
- net SDA: track 132.8 -> 146.1 mm
- net VCC: track 123.1 -> 135.7 mm, vias 3 -> 2
- net GND: track 0.00 -> 7.72 mm
- net INT0: track 82.7 -> 89.8 mm
- net OC1A: track 100.8 -> 104.7 mm
Other:
- outline, holes or cut-outs redrawn
