File: Electronic/Placa PCB/v2/interstage_A2v2.sch (EAGLE design)
At the start: 7 parts, among them Q1 PMV16XNR, U1 MCP9808T-E/MS, U3 MCP9808T-E/MS

Commit message: Placas PCB
Parts:
- removed I2C_PLACAS/I2C_OBC1: 53261-0871, SamacSys_Parts:53261-0871
- removed R5, R9: 330 Ohm, rcl:R-EU_R1206
- added CONEXION_B2: 53261-7006, SamacSys_Parts:53261-7006
- added PINES_SWITCH: (no value), con-lstb:MA03-1
- added R_MOSFET, R_SWITCH: ERA-8AEB331V, resistor_330_smd:ERA-8AEB331V
- renumbered I2C_PLACAS/I2C_OBC to CONEXION_B1, U1 to T5, U3 to T6
Connections:
- net MOSFET renamed NICROMO
- removed net N$4: R9.1
- new net N$7: PINES_SWITCH.3
- net AIN0: now also R_MOSFET.1; no longer R5.2
- net GND: now also CONEXION_B2.5, R_MOSFET.2, R_SWITCH.1, T5.A0, T5.A1, T6.A1; no longer I2C_PLACAS/I2C_OBC1.7, R5.1
- net INT0: now also CONEXION_B2.2; no longer I2C_PLACAS/I2C_OBC1.4
- net OC1A: now also CONEXION_B2.1; no longer I2C_PLACAS/I2C_OBC1.3
- net SCL: now also CONEXION_B2.4; no longer I2C_PLACAS/I2C_OBC1.6
- net SDA: now also CONEXION_B2.3; no longer I2C_PLACAS/I2C_OBC1.5
- net T0: now also PINES_SWITCH.2, R_SWITCH.2; no longer R9.2
- net VCC: now also CONEXION_B2.6, PINES_SWITCH.1, T5.A2, T6.A0, T6.A2; no longer I2C_PLACAS/I2C_OBC1.8
