File: Electronic/Placa PCB/v2/interstage_B1v2.brd (EAGLE design)
At the start: 82.5 x 29 mm, 8 parts, among them J1 0532611271, Q1 PMV16XNR, U1 LM70CIMM-3, U2 LM70CIMM-3

Commit message: Avance
Parts:
- removed C1, C2: 0.1pF, rcl:C0603K
- removed J1: 0532611271, picoblade:MOLEX_0532611271
- removed R7: 330 Ohm, rcl:R1206
- removed U2: LM70CIMM-3, LM70CIMM-3:SOP65P490X110-8N
- added I2C_PLACAS/I2C_OBC, I2C_PLACAS/I2C_OBC1: 53261-0871, SamacSys_Parts:53261-0871
- added R9: 330 Ohm, rcl:R1206
- added U3: MCP9808T-E/MS, sensorSPEL:SOP65P490X110-8N
- U1: value LM70CIMM-3 -> MCP9808T-E/MS; device LM70CIMM-3:SOP65P490X110-8N -> sensorSPEL:SOP65P490X110-8N
- moved U1 23.8 mm to (21.0, 20.0)
- moved R5 16.6 mm to (17.0, 12.5)
- moved Q1 12.4 mm to (25.1, 8.70), turned to 90 degrees
Connections:
- removed net MISO: J1.4, U1.1, U2.1
- removed net MOSI: J1.5, U1.7, U2.7
- removed net N$1: R7.1
- removed net SCK: J1.3, U1.2, U2.2
- new net N$4: R9.1
- new net SCL: I2C_PLACAS/I2C_OBC1.6, U1.2, U3.2
- new net SDA: I2C_PLACAS/I2C_OBC1.5, U1.1, U3.1
- net AIN0: now also I2C_PLACAS/I2C_OBC.5, I2C_PLACAS/I2C_OBC1.3; no longer J1.8
- net AIN1: now also I2C_PLACAS/I2C_OBC.4, R9.2; no longer J1.7
- net GND: now also I2C_PLACAS/I2C_OBC.2, I2C_PLACAS/I2C_OBC1.7, U3.4; no longer C1.2, C2.2, J1.2, U2.4
- net INT0: now also I2C_PLACAS/I2C_OBC.7, I2C_PLACAS/I2C_OBC1.2; no longer J1.10, R7.2
- net OC1A: now also I2C_PLACAS/I2C_OBC.3, I2C_PLACAS/I2C_OBC1.4; no longer J1.6, Q1.1, R5.2
- net T0: now also I2C_PLACAS/I2C_OBC1.1; no longer J1.11
- net T1: now also I2C_PLACAS/I2C_OBC.6, Q1.1, R5.2; no longer J1.9
- net VCC: now also I2C_PLACAS/I2C_OBC.1, I2C_PLACAS/I2C_OBC1.8, U1.8, U3.8; no longer C1.1, C2.1, J1.1, U1.5, U2.5
Routing:
- net AIN0: track 0.00 -> 88.6 mm
- net MISO: track 81.6 -> 0.00 mm, vias 1 -> 0
- net OC1A: track 24.3 -> 97.4 mm
- net SDA: track 0.00 -> 67.4 mm, vias 0 -> 2
- net SCK: track 65.4 -> 0.00 mm, vias 1 -> 0
- net SCL: track 0.00 -> 64.6 mm, vias 0 -> 2
- net INT0: track 4.79 -> 58.8 mm
- net MOSI: track 42.5 -> 0.00 mm, vias 1 -> 0
- net T1: track 0.00 -> 25.1 mm
- net VCC: track 66.8 -> 76.9 mm, vias 1 -> 3
- net GND: track 8.01 -> 0.00 mm
- net AIN1: track 0.00 -> 4.63 mm
- net MOSFET: track 5.50 -> 4.73 mm
Other:
- outline, holes or cut-outs redrawn

Commit message: Placas PCB
Parts:
- removed I2C_PLACAS/I2C_OBC: 53261-0871, SamacSys_Parts:53261-0871
- removed R5, R9: 330 Ohm, rcl:R1206
- added CONEXION_A1: 53261-0871, SamacSys_Parts:53261-0871
- added R_MOSFET, R_SWITCH: ERA-8AEB331V, resistor_330_smd:RESC3216X70N
- added SV1: (no value), con-lstb:MA03-1
- moved Q1 21.7 mm to (46.0, 14.5), turned to 180 degrees
- renumbered I2C_PLACAS/I2C_OBC1 to CONEXION_A2, U1 to T3, U3 to T4
Connections:
- net MOSFET renamed NICROMO
- removed net N$4: R9.1
- net AIN0: now also CONEXION_A1.5; no longer I2C_PLACAS/I2C_OBC.5
- net AIN1: now also CONEXION_A1.4, R_SWITCH.2, SV1.2; no longer I2C_PLACAS/I2C_OBC.4, R9.2
- net GND: now also CONEXION_A1.2, R_MOSFET.2, R_SWITCH.1, T3.5, T3.7, T4.5; no longer I2C_PLACAS/I2C_OBC.2, R5.1
- net INT0: now also CONEXION_A1.7; no longer I2C_PLACAS/I2C_OBC.7
- net OC1A: now also CONEXION_A1.3; no longer I2C_PLACAS/I2C_OBC.3
- net T0: now also CONEXION_A1.8
- net T1: now also CONEXION_A1.6, R_MOSFET.1; no longer I2C_PLACAS/I2C_OBC.6, R5.2
- net VCC: now also CONEXION_A1.1, SV1.1, T3.6, T4.6, T4.7; no longer I2C_PLACAS/I2C_OBC.1
Routing:
- net T0: track 0.00 -> 56.2 mm
- net VCC: track 76.9 -> 124.0 mm, vias 3 -> 2
- net T1: track 25.1 -> 55.6 mm
- net AIN1: track 4.63 -> 30.6 mm, vias 0 -> 1
- net AIN0: track 88.6 -> 75.0 mm, vias 0 -> 2
- net OC1A: track 97.4 -> 88.6 mm
- net GND: track 0.00 -> 5.75 mm
- net SCL: track 64.6 -> 60.7 mm, vias 2 -> 1
- net INT0: track 58.8 -> 56.3 mm
- net SDA: track 67.4 -> 67.5 mm, vias 2 -> 1
Other:
- outline, holes or cut-outs redrawn
