File: Electronic/Placa PCB/v2/interstage_B1v2.sch (EAGLE design)
At the start: 7 parts, among them Q1 PMV16XNR, U1 MCP9808T-E/MS, U3 MCP9808T-E/MS

Commit message: Placas PCB
Parts:
- removed I2C_PLACAS/I2C_OBC, I2C_PLACAS/I2C_OBC1: 53261-0871, SamacSys_Parts:53261-0871
- removed R5, R9: 330 Ohm, rcl:R-EU_R1206
- added CONEXION_A1, CONEXION_A2: 53261-0871, SamacSys_Parts:53261-0871
- added R_MOSFET, R_SWITCH: ERA-8AEB331V, resistor_330_smd:ERA-8AEB331V
- added SV1: (no value), con-lstb:MA03-1
- renumbered U1 to T3, U3 to T4
Connections:
- net MOSFET renamed NICROMO
- removed net N$4: R9.1
- net AIN0: now also CONEXION_A1.5, CONEXION_A2.3; no longer I2C_PLACAS/I2C_OBC.5, I2C_PLACAS/I2C_OBC1.3
- net AIN1: now also CONEXION_A1.4, R_SWITCH.2, SV1.2; no longer I2C_PLACAS/I2C_OBC.4, R9.2
- net GND: now also CONEXION_A1.2, CONEXION_A2.7, R_MOSFET.2, R_SWITCH.1, T3.A0, T3.A2, T4.A2; no longer I2C_PLACAS/I2C_OBC.2, I2C_PLACAS/I2C_OBC1.7, R5.1
- net INT0: now also CONEXION_A1.7, CONEXION_A2.2; no longer I2C_PLACAS/I2C_OBC.7, I2C_PLACAS/I2C_OBC1.2
- net OC1A: now also CONEXION_A1.3, CONEXION_A2.4; no longer I2C_PLACAS/I2C_OBC.3, I2C_PLACAS/I2C_OBC1.4
- net SCL: now also CONEXION_A2.6; no longer I2C_PLACAS/I2C_OBC1.6
- net SDA: now also CONEXION_A2.5; no longer I2C_PLACAS/I2C_OBC1.5
- net T0: now also CONEXION_A1.8, CONEXION_A2.1; no longer I2C_PLACAS/I2C_OBC1.1
- net T1: now also CONEXION_A1.6, R_MOSFET.1; no longer I2C_PLACAS/I2C_OBC.6, R5.2
- net VCC: now also CONEXION_A1.1, CONEXION_A2.8, SV1.1, T3.A1, T4.A0, T4.A1; no longer I2C_PLACAS/I2C_OBC.1, I2C_PLACAS/I2C_OBC1.8
