File: Electronic/Placa PCB/v2/interstage_mini.brd (EAGLE design)
At the start: 13 x 10.1 mm, 2 parts

Commit message: Mini placas
Parts:
- removed S1: D3SH-A1L, D3SH-A1L:SW_D3SH-A1L
- added U$2: SWITCH, SWITCH:SWITCH
Connections:
- new net NC: U$1.NC, U$2.NC
- net NO: now also U$2.NO; no longer S1.2
- net VCC: now also U$2.VCC; no longer S1.1
Routing:
- net NO: track 7.49 -> 2.97 mm
- net VCC: track 6.78 -> 2.97 mm
- net NC: track 0.00 -> 2.97 mm
Changed lines of the file:
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@@
 <?xml version="1.0" encoding="utf-8"?>
 <!DOCTYPE eagle SYSTEM "eagle.dtd">
-<eagle version="9.6.1">
+<eagle version="9.2.2">
 <drawing>
 <settings>
@@
 </autorouter>
 <elements>
-<element name="S1" library="D3SH-A1L" package="SW_D3SH-A1L" value="D3SH-A1L" x="6.5" y="7.91" smashed="yes">
-<attribute name="ARROW_PURCHASE_URL" value="" x="6.5" y="7.91" size="1.778" layer="27" font="vector" display="off"/>
-<attribute name="DESCRIPTION" value=" Switch SPST-NO Surface Mount, Right Angle " x="6.5" y="7.91" size="1.778" layer="27" font="vector" display="off"/>
-<attribute name="MF" value="Omron" x="6.5" y="7.91" size="1.778" layer="27" font="vector" display="off"/>
-<attribute name="MP" value="D3SH-A1L" x="6.5" y="7.91" size="1.778" layer="27" font="vector" display="off"/>
-<attribute name="NAME" x="3.99901875" y="5.909209375" size="1.2705" layer="25" rot="R90"/>
-<attribute name="PACKAGE" value="None" x="6.5" y="7.91" size="1.778" layer="27" font="vector" display="off"/>
-<attribute name="VALUE" x="10.25713125" y="5.9062" size="1.272409375" layer="27" rot="R90"/>
-</element>
 <element name="U$1" library="conector" package="CONECTOR" value="CONECTOR" x="6.5" y="0" smashed="yes"/>
+<element name="U$2" library="SWITCH" package="SWITCH" value="SWITCH" x="6.5" y="3.97" smashed="yes"/>
 </elements>
 <signals>
 <signal name="VCC">
-<contactref element="S1" pad="1"/>
 <contactref element="U$1" pad="VCC"/>
-<wire x1="3.96" y1="2" x2="3.96" y2="7.89" width="0.5" layer="1"/>
-<wire x1="3.96" y1="7.89" x2="4.85" y2="7.91" width="0.5" layer="1"/>
+<contactref element="U$2" pad="VCC"/>
+<wire x1="3.96" y1="1" x2="3.96" y2="3.97" width="0.5" layer="1"/>
 </signal>
 <signal name="NO">
-<contactref element="S1" pad="2"/>
 <contactref element="U$1" pad="NO"/>
-<wire x1="6.5" y1="2" x2="6.5" y2="5.5" width="0.5" layer="1"/>
-<wire x1="6.5" y1="5.5" x2="8.15" y2="5.5" width="0.5" layer="1"/>
-<wire x1="8.15" y1="5.5" x2="8.15" y2="7.835" width="0.5" layer="1"/>
+<contactref element="U$2" pad="NO"/>
+<wire x1="6.5" y1="1" x2="6.5" y2="3.97" width="0.5" layer="1"/>
+</signal>
+<signal name="NC">
+<contactref element="U$1" pad="NC"/>
+<contactref element="U$2" pad="NC"/>
+<wire x1="9.04" y1="1" x2="9.04" y2="3.97" width="0.5" layer="1"/>
 </signal>
 </signals>

Commit message: Presentacion II
Changed lines of the file:
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@@
 <contactref element="U$1" pad="VCC"/>
 <contactref element="U$2" pad="VCC"/>
-<wire x1="3.96" y1="1" x2="3.96" y2="3.97" width="0.5" layer="1"/>
+<wire x1="3.96" y1="1" x2="3.96" y2="3.97" width="1" layer="1"/>
 </signal>
 <signal name="NO">
 <contactref element="U$1" pad="NO"/>
 <contactref element="U$2" pad="NO"/>
-<wire x1="6.5" y1="1" x2="6.5" y2="3.97" width="0.5" layer="1"/>
+<wire x1="6.5" y1="1" x2="6.5" y2="3.97" width="1" layer="1"/>
 </signal>
 <signal name="NC">
 <contactref element="U$1" pad="NC"/>
 <contactref element="U$2" pad="NC"/>
-<wire x1="9.04" y1="1" x2="9.04" y2="3.97" width="0.5" layer="1"/>
+<wire x1="9.04" y1="1" x2="9.04" y2="3.97" width="1" layer="1"/>
 </signal>
 </signals>
