File: Electronic/Placa PCB/v2/interstage_mini.sch (EAGLE design)
At the start: 2 parts

Commit message: Mini placas
Parts:
- removed S1: D3SH-A1L, D3SH-A1L:D3SH-A1L
- added U$2: SWITCH, SWITCH:SWITCH
Connections:
- new net NC: U$1.NC, U$2.NC
- net NO: now also U$2.NO; no longer S1.NO
- net VCC: now also U$2.VCC; no longer S1.COM
Changed lines of the file:
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@@
 </classes>
 <parts>
-<part name="S1" library="D3SH-A1L" deviceset="D3SH-A1L" device=""/>
 <part name="U$1" library="conector" deviceset="CONECTOR" device=""/>
+<part name="U$2" library="SWITCH" deviceset="SWITCH" device=""/>
 </parts>
 <sheets>
@@
 </plain>
 <instances>
-<instance part="S1" gate="G$1" x="60.96" y="60.96" smashed="yes">
-<attribute name="NAME" x="53.334040625" y="73.6699" size="1.779390625" layer="95"/>
-<attribute name="VALUE" x="53.32735" y="50.7831" size="1.78095" layer="96"/>
-</instance>
-<instance part="U$1" gate="G$1" x="60.96" y="27.94" smashed="yes"/>
+<instance part="U$1" gate="G$1" x="0" y="10.16" smashed="yes"/>
+<instance part="U$2" gate="G$1" x="0" y="40.64" smashed="yes"/>
 </instances>
 <busses>
@@
 <net name="VCC" class="0">
 <segment>
-<pinref part="S1" gate="G$1" pin="COM"/>
-<wire x1="48.26" y1="60.96" x2="43.18" y2="60.96" width="0.1524" layer="91"/>
-<label x="43.18" y="60.96" size="1.778" layer="95" rot="R180" xref="yes"/>
+<pinref part="U$1" gate="G$1" pin="VCC"/>
+<wire x1="-5.08" y1="15.24" x2="-5.08" y2="17.78" width="0.1524" layer="91"/>
+<label x="-5.08" y="17.78" size="1.778" layer="95" rot="R90" xref="yes"/>
 </segment>
 <segment>
-<pinref part="U$1" gate="G$1" pin="VCC"/>
-<wire x1="55.88" y1="33.02" x2="55.88" y2="38.1" width="0.1524" layer="91"/>
-<label x="55.88" y="38.1" size="1.778" layer="95" rot="R90" xref="yes"/>
+<pinref part="U$2" gate="G$1" pin="VCC"/>
+<wire x1="-5.08" y1="45.72" x2="-5.08" y2="50.8" width="0.1524" layer="91"/>
+<label x="-5.08" y="50.8" size="1.778" layer="95" rot="R90" xref="yes"/>
 </segment>
 </net>
 <net name="NO" class="0">
 <segment>
-<pinref part="S1" gate="G$1" pin="NO"/>
-<wire x1="73.66" y1="60.96" x2="78.74" y2="60.96" width="0.1524" layer="91"/>
-<label x="78.74" y="60.96" size="1.778" layer="95" xref="yes"/>
+<pinref part="U$1" gate="G$1" pin="NO"/>
+<wire x1="0" y1="15.24" x2="0" y2="17.78" width="0.1524" layer="91"/>
+<label x="0" y="17.78" size="1.778" layer="95" rot="R90" xref="yes"/>
 </segment>
 <segment>
-<pinref part="U$1" gate="G$1" pin="NO"/>
-<wire x1="60.96" y1="33.02" x2="60.96" y2="38.1" width="0.1524" layer="91"/>
-<label x="60.96" y="38.1" size="1.778" layer="95" rot="R90" xref="yes"/>
+<pinref part="U$2" gate="G$1" pin="NO"/>
+<wire x1="0" y1="45.72" x2="0" y2="50.8" width="0.1524" layer="91"/>
+<label x="0" y="50.8" size="1.778" layer="95" rot="R90" xref="yes"/>
 </segment>
 </net>
+<net name="NC" class="0">
+<segment>
+<pinref part="U$1" gate="G$1" pin="NC"/>
+<wire x1="5.08" y1="15.24" x2="5.08" y2="17.78" width="0.1524" layer="91"/>
+<label x="5.08" y="17.78" size="1.778" layer="95" rot="R90" xref="yes"/>
+</segment>
+<segment>
+<pinref part="U$2" gate="G$1" pin="NC"/>
+<wire x1="5.08" y1="45.72" x2="5.08" y2="50.8" width="0.1524" layer="91"/>
+<label x="5.08" y="50.8" size="1.778" layer="95" rot="R90" xref="yes"/>
+</segment>
+</net>
