File: Electronic/Placa PCB/v2/interstage_miniSMD.brd (EAGLE design)
At the start: 13 x 10.1 mm, 2 parts

Commit message: Presentacion II
Routing:
- net NO: track 8.46 -> 7.50 mm
- net VCC: track 7.78 -> 7.26 mm
Changed lines of the file:
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@@
 <signal name="VCC">
 <contactref element="S1" pad="1"/>
-<wire x1="3.96" y1="7.89" x2="4.85" y2="7.89" width="0.5" layer="1"/>
 <contactref element="U$1" pad="VCC"/>
-<wire x1="3.96" y1="1" x2="3.96" y2="7.89" width="0.5" layer="1"/>
+<wire x1="3.96" y1="4.5" x2="3.96" y2="1" width="1" layer="1"/>
+<wire x1="4.85" y1="7.89" x2="4.85" y2="5.39" width="1" layer="1"/>
+<wire x1="4.85" y1="5.39" x2="3.96" y2="4.5" width="1" layer="1"/>
 </signal>
 <signal name="NO">
 <contactref element="S1" pad="2"/>
-<wire x1="6.5" y1="5.5" x2="8.15" y2="5.5" width="0.5" layer="1"/>
-<wire x1="8.15" y1="5.5" x2="8.15" y2="7.815" width="0.5" layer="1"/>
+<wire x1="8.15" y1="7.815" x2="8.15" y2="5.5" width="1" layer="1"/>
 <contactref element="U$1" pad="NO"/>
-<wire x1="6.5" y1="1" x2="6.5" y2="5.5" width="0.5" layer="1"/>
+<wire x1="8.15" y1="5.5" x2="6.5" y2="3.85" width="1" layer="1"/>
+<wire x1="6.5" y1="3.85" x2="6.5" y2="1" width="1" layer="1"/>
 </signal>
 </signals>
