File: Electronic/Placa PCB/v2/interstage_A2.brd (EAGLE design)
At the start: 82.5 x 29 mm, 8 parts, among them Q1 PMV16XNR, T5 MCP9808T-E/MS, T6 MCP9808T-E/MS

Commit message: gerbers
Parts:
- R1, R2: value ERA-8AEB331V -> 330
- renumbered CONEXION_B1 to J1, CONEXION_B2 to J2, PINES_SWITCH to J3, Q1 to M1, R_MOSFET to R1, R_SWITCH to R2
Routing:
- net INT0: track 82.9 -> 81.7 mm
